Commit message: updates

File: burg-toolkit/data/gripper/dummy_xyz_robot.urdf (robot description, URDF)
Before this commit: robot dummy_robot, 7 links, 6 joints
Links:
- removed link pitch_control
- removed link roll_control
- removed link yaw_control
Joints:
- removed joint gripper_pitch
- removed joint gripper_roll
- removed joint gripper_yaw
- joint center_z: child yaw_control -> end_effector_link
